Commit message: finished task 2

File: Step2/table_macro.xacro (robot description, xacro)
@@ -4,10 +4,10 @@
     <!-- Constants for robot dimensions -->
     <xacro:property name="table_width" value="1" />
-    <xacro:property name="table_length" value = "2"/>
+    <xacro:property name="table_length" value = "1"/>
     <xacro:property name="table_height" value = "1"/>
-    <xacro:property name="table_thickness" value = "0.05"/>
-    <xacro:property name="leg_length" value="{table_height - table_thickness" /> <!-- base_link -->
+    <xacro:property name="table_thickness" value = "0.1"/>
+    <xacro:property name="leg_length" value="${table_height - table_thickness}" /> <!-- base_link -->
     <xacro:property name="leg_radius" value="0.05" /> <!-- link1 -->
-    <joint name="${prefix}top" type="fixed">
+    <joint name="${prefix}top_joint" type="fixed">
       <xacro:insert_block name="origin" />
       <parent link="${parent}" />
@@ -17,15 +17,15 @@
     <link name="${prefix}top">
       <visual>
-        <origin xyz="0 0 ${table_height}" rpy="0 0 0" />
+        <origin xyz="0 0 ${- table_thickness/2}" rpy="0 0 0" />
         <geometry>
-          <box size="${table_length} ${table_width} ${table_thickness}" />
+          <box size="${table_length} ${table_width} ${table_thickness }" />
         </geometry>
         <material name="brown" />
       </visual>
     </link>
-    <joint name="${prefix}leg1" type="continuous">
+    <joint name="${prefix}joint1" type="fixed">
       <parent link="${prefix}top" />
       <child link="${prefix}leg1" />
-      <origin xyz="0 ${width} ${height0 - axel_offset}" rpy="0 0 0" />
+      <origin xyz = "${table_length / 2 - leg_radius} ${table_width / 2 - leg_radius} ${(table_height -table_thickness) - table_height} " rpy = "0 0 0"/>
       <axis xyz="0 1 0" />
     </joint>
@@ -33,7 +33,55 @@
     <link name="${prefix}leg1">
       <visual>
-        <origin xyz="${table_height/2} ${table_width/2} ${height1/2 - axel_offset}" rpy="0 0 0" />
+        <origin xyz="0 0 ${(- table_height + table_thickness)/2 }" rpy="0 0 0" />
         <geometry>
-          <box size="${width} ${width} ${height1}" />
+          <box size="${leg_radius} ${leg_radius} ${leg_length}" />
+        </geometry>
+        <material name="light_grey" />
+      </visual>
+    </link>
+    <!-- Leg2  -->
+    <joint name="${prefix}joint2" type="fixed">
+      <parent link="${prefix}top" />
+      <child link="${prefix}leg2" />
+       <origin xyz = "${-(table_length / 2 - leg_radius)} ${table_width / 2 - leg_radius} ${(table_height -table_thickness) -1}" rpy = "0 0 0"/>
+      <axis xyz="0 1 0" />
+    </joint>
+    <link name="${prefix}leg2">
+      <visual>
+        <origin xyz="0 0 ${(- table_height + table_thickness)/2}" rpy="0 0 0" />
+        <geometry>
+          <box size="${leg_radius} ${leg_radius} ${leg_length}" />
+        </geometry>
+        <material name="light_grey" />
+      </visual>
+    </link>
+    <!-- Leg3  -->
+    <joint name="${prefix}joint3" type="fixed">
+      <parent link="${prefix}top" />
+      <child link="${prefix}leg3" />
+       <origin xyz = "${-(table_length / 2 - leg_radius)} ${-(table_width / 2 - leg_radius)} ${(table_height -table_thickness) - 1}" rpy = "0 0 0"/>
+      <axis xyz="0 1 0" />
+    </joint>
+    <link name="${prefix}leg3">
+      <visual>
+        <origin xyz="0 0 ${(- table_height + table_thickness)/2}" rpy="0 0 0" />
+        <geometry>
+          <box size="${leg_radius} ${leg_radius} ${leg_length}" />
+        </geometry>
+        <material name="light_grey" />
+      </visual>
+    </link>
+    <!-- Leg4  -->
+    <joint name="${prefix}joint4" type="fixed">
+      <parent link="${prefix}top" />
+      <child link="${prefix}leg4" />
+       <origin xyz = "${table_length / 2 - leg_radius} ${-(table_width / 2 - leg_radius)} ${(table_height -table_thickness) -1}" rpy = "0 0 0"/>
+      <axis xyz="0 1 0" />
+    </joint>
+    <link name="${prefix}leg4">
+      <visual>
+        <origin xyz="0 0 ${(- table_height + table_thickness)/2}" rpy="0 0 0" />
+        <geometry>
+          <box size="${leg_radius} ${leg_radius} ${leg_length}" />
         </geometry>
         <material name="light_grey" />
