Commit message: done :)

File: ws2/src/table_description/urdf/table_macro.xacro (robot description, xacro)
@@ -17,5 +17,5 @@
     <link name="${prefix}top">
       <visual>
-        <origin xyz="0 0 0" rpy="0 0 0" />
+        <origin xyz="0 0 ${-table_thickness/2}" rpy="0 0 0" />
         <geometry>
           <box size="${table_length} ${table_width} ${table_thickness }" />
